Commit message: All new files pushed

File: urdf/walle.urdf (robot description, URDF)
Before this commit: robot wallewithoutpcb1.SLDASM, 9 links, 8 joints
Links:
- removed link backleftspacers
- removed link backrightspacers
- removed link frontdir
- removed link frontleftspacers
- removed link frontrightspacers
- removed link pcb
- link chassis: mass 0.0914673846752495 -> 0.276711529585972; geometry collision mesh filename=package://walle/meshes/chassis.STL; visual mesh filename=package://walle/meshes/chassis.STL
- link leftwheel: mass 0.0607932288876856 -> 0.0297341396000603; geometry collision mesh filename=package://walle/meshes/leftwheel.STL; visual mesh filename=package://walle/meshes/leftwheel.STL
- link rightwheel: mass 0.0607932288876853 -> 0.02973413960006; geometry collision mesh filename=package://walle/meshes/rightwheel.STL; visual mesh filename=package://walle/meshes/rightwheel.STL
Joints:
- removed joint bls
- removed joint brs
- removed joint fd
- removed joint fls
- removed joint frs
- removed joint pcb

Commit message: Files for bot created on 22nd September are uploaded

File: urdf/walle.urdf (robot description, URDF)
Before this commit: robot walle, 3 links, 2 joints
Links:
- link chassis: mass 0.276711529585972 -> 0.280599674625568; geometry collision mesh filename=package://wallh/meshes/chassis.STL; visual mesh filename=package://wallh/meshes/chassis.STL
- link leftwheel: mass 0.0297341396000603 -> 0.0297341396000601; geometry collision mesh filename=package://wallh/meshes/leftwheel.STL; visual mesh filename=package://wallh/meshes/leftwheel.STL
- link rightwheel: mass 0.02973413960006 -> 0.0297341396000606; geometry collision mesh filename=package://wallh/meshes/rightwheel.STL; visual mesh filename=package://wallh/meshes/rightwheel.STL
Joints:
- joint lw: limit lower=0 upper=0 effort=1 velocity=1 -> lower=0 upper=0 effort=100 velocity=100; origin xyz=-0.09295 -0.014082 -0.018804 rpy=0 0 0 -> xyz=-0.06625 -0.014071 -0.018803 rpy=0 0 0
- joint rw: limit lower=0 upper=0 effort=1 velocity=1 -> lower=0 upper=0 effort=100 velocity=100; origin xyz=0.09295 -0.014082 -0.018802 rpy=0 0 0 -> xyz=0.06625 -0.014071 -0.018803 rpy=0 0 0

Commit message: Uploaded on 23rd september 11:56 pm

File: urdf/walle.urdf (robot description, URDF)
Before this commit: robot wallh, 3 links, 2 joints
Links:
- added link leftshaft, mass 0.00040732; collision mesh filename=package://ab/meshes/leftshaft.STL; visual mesh filename=package://ab/meshes/leftshaft.STL
- added link rightshaft, mass 0.00040732; collision mesh filename=package://ab/meshes/rightshaft.STL; visual mesh filename=package://ab/meshes/rightshaft.STL
- link chassis: mass 0.280599674625568 -> 5; geometry collision mesh filename=package://ab/meshes/chassis.STL; visual mesh filename=package://ab/meshes/chassis.STL
- link leftwheel: mass 0.0297341396000601 -> 0.29734; geometry collision mesh filename=package://ab/meshes/leftwheel.STL; visual mesh filename=package://ab/meshes/leftwheel.STL
- link rightwheel: mass 0.0297341396000606 -> 0.29734; geometry collision mesh filename=package://ab/meshes/rightwheel.STL; visual mesh filename=package://ab/meshes/rightwheel.STL
Joints:
- added joint ls: type revolute, parent chassis, child leftshaft, origin xyz=-0.06675 -0.014071 -0.018803 rpy=0 0 0, axis -1 0 0, limit lower=0 upper=0 effort=1000 velocity=1000
- added joint rs: type revolute, parent chassis, child rightshaft, origin xyz=0.06675 -0.014071 -0.018803 rpy=0 0 0, axis -1 0 0, limit lower=0 upper=0 effort=1000 velocity=1000
- joint lw: limit lower=0 upper=0 effort=100 velocity=100 -> lower=0 upper=0 effort=1000 velocity=1000; origin xyz=-0.06625 -0.014071 -0.018803 rpy=0 0 0 -> xyz=0 0 0 rpy=0 0 0; parent chassis -> leftshaft
- joint rw: limit lower=0 upper=0 effort=100 velocity=100 -> lower=0 upper=0 effort=1000 velocity=1000; origin xyz=0.06625 -0.014071 -0.018803 rpy=0 0 0 -> xyz=0 0 0 rpy=0 0 0; parent chassis -> rightshaft

Commit message: All bot files for the latest version of the bot

File: urdf/walle.urdf (robot description, URDF)
Before this commit: robot ab, 5 links, 4 joints
Links:
- link chassis: geometry collision mesh filename=package://a/meshes/chassis.STL; visual mesh filename=package://a/meshes/chassis.STL
- link leftshaft: mass 0.00040732 -> 0.1; geometry collision mesh filename=package://a/meshes/leftshaft.STL; visual mesh filename=package://a/meshes/leftshaft.STL
- link leftwheel: mass 0.29734 -> 0.4; geometry collision mesh filename=package://a/meshes/leftwheel.STL; visual mesh filename=package://a/meshes/leftwheel.STL
- link rightshaft: mass 0.00040732 -> 0.1; geometry collision mesh filename=package://a/meshes/rightshaft.STL; visual mesh filename=package://a/meshes/rightshaft.STL
- link rightwheel: mass 0.29734 -> 0.4; geometry collision mesh filename=package://a/meshes/rightwheel.STL; visual mesh filename=package://a/meshes/rightwheel.STL
Joints:
- joint lw: origin xyz=0 0 0 rpy=0 0 0 -> xyz=-0.0103 -0.0011117 0.0011507 rpy=0 0 0
- joint rw: origin xyz=0 0 0 rpy=0 0 0 -> xyz=0.0090108 0 0 rpy=0 0 0

Commit message: Files added after meet

File: urdf/walle.urdf (robot description, URDF)
Before this commit: robot a, 5 links, 4 joints
Links:
- link chassis: mass 5 -> 0.75; geometry collision mesh filename=package://aaa/meshes/chassis.STL; visual mesh filename=package://aaa/meshes/chassis.STL
- link leftshaft: mass 0.1 -> 0.005; geometry collision mesh filename=package://aaa/meshes/leftshaft.STL; visual mesh filename=package://aaa/meshes/leftshaft.STL
- link leftwheel: mass 0.4 -> 0.03; geometry collision mesh filename=package://aaa/meshes/leftwheel.STL; visual mesh filename=package://aaa/meshes/leftwheel.STL
- link rightshaft: mass 0.1 -> 0.005; geometry collision mesh filename=package://aaa/meshes/rightshaft.STL; visual mesh filename=package://aaa/meshes/rightshaft.STL
- link rightwheel: mass 0.4 -> 0.03; geometry collision mesh filename=package://aaa/meshes/rightwheel.STL; visual mesh filename=package://aaa/meshes/rightwheel.STL
Joints:
- joint ls: origin xyz=-0.06675 -0.014071 -0.018803 rpy=0 0 0 -> xyz=-0.06575 -0.014071 -0.018803 rpy=0 0 0
- joint lw: origin xyz=-0.0103 -0.0011117 0.0011507 rpy=0 0 0 -> xyz=-0.0216 0 0 rpy=0 0 0
- joint rs: axis -1 0 0 -> 1 0 0; origin xyz=0.06675 -0.014071 -0.018803 rpy=0 0 0 -> xyz=0.06575 -0.014071 -0.018803 rpy=0 0 0
- joint rw: axis -1 0 0 -> 1 0 0; origin xyz=0.0090108 0 0 rpy=0 0 0 -> xyz=0.0216 0 0 rpy=0 0 0

Commit message: Latest files added

File: urdf/walle.urdf (robot description, URDF)
Before this commit: robot aaa, 5 links, 4 joints
Links:
- removed link chassis
- removed link leftshaft
- removed link leftwheel
- removed link rightshaft
- removed link rightwheel
- added link base_link, mass 0.0915522076768964; collision mesh filename=meshes/base_link.STL; visual mesh filename=meshes/base_link.STL
- added link camera_link; collision box size=0.01 0.01 0.01; visual box size=0.01 0.01 0.01
- added link imu_link; collision box size=0.001 0.001 0.001; visual box size=0.001 0.001 0.001
- added link leftlink, mass 0.0297341394891575; collision mesh filename=meshes/leftlink.STL; visual mesh filename=meshes/leftlink.STL
- added link rightlink, mass 0.0297341394891515; collision mesh filename=meshes/rightlink.STL; visual mesh filename=meshes/rightlink.STL
Joints:
- removed joint ls
- removed joint lw
- removed joint rs
- removed joint rw
- added joint camera_joint: type fixed, parent base_link, child camera_link, origin xyz=0 0 0
- added joint imu_joint: type fixed, parent base_link, child imu_link, origin xyz=0 0 0.01
- added joint leftjoint: type continuous, parent base_link, child leftlink, origin xyz=-0.0054501 0.10601 -0.017901 rpy=0 0 0, axis 0 1 0, limit effort=1 velocity=1
- added joint rightjoint: type continuous, parent base_link, child rightlink, origin xyz=-0.0063446 -0.10601 -0.017901 rpy=0 0 0, axis 0 1 0, limit effort=1 velocity=1
